Commit message: updated hw handler

File: hardware-handler/nightmare_description/urdf/nightmare.xacro (robot description, xacro)
@@ -24,5 +24,5 @@
   </collision>
 </link>
-<link name="leg_2_coxa_1">
+<link name="leg_3_coxa_1">
   <inertial>
     <origin rpy="0 0 0" xyz="0.024052035496447563 -0.024052034022785593 -0.02050000171122137"/>
@@ -33,5 +33,5 @@
     <origin rpy="0 0 0" xyz="-0.068335 0.078335 -0.0385"/>
     <geometry>
-      <mesh filename="package://nightmare_description/meshes/leg_2_coxa_1.stl" scale="0.001 0.001 0.001"/>
+      <mesh filename="package://nightmare_description/meshes/leg_3_coxa_1.stl" scale="0.001 0.001 0.001"/>
     </geometry>
     <material name="silver"/>
@@ -40,9 +40,9 @@
     <origin rpy="0 0 0" xyz="-0.068335 0.078335 -0.0385"/>
     <geometry>
-      <mesh filename="package://nightmare_description/meshes/leg_2_coxa_1.stl" scale="0.001 0.001 0.001"/>
-    </geometry>
-  </collision>
-</link>
-<link name="leg_3_coxa_1">
+      <mesh filename="package://nightmare_description/meshes/leg_3_coxa_1.stl" scale="0.001 0.001 0.001"/>
+    </geometry>
+  </collision>
+</link>
+<link name="leg_2_coxa_1">
   <inertial>
     <origin rpy="0 0 0" xyz="0.03401538718261085 9.93696248999688e-10 -0.02050000171212193"/>
@@ -53,5 +53,5 @@
     <origin rpy="0 0 0" xyz="-0.093 -0.0 -0.0385"/>
     <geometry>
-      <mesh filename="package://nightmare_description/meshes/leg_3_coxa_1.stl" scale="0.001 0.001 0.001"/>
+      <mesh filename="package://nightmare_description/meshes/leg_2_coxa_1.stl" scale="0.001 0.001 0.001"/>
     </geometry>
     <material name="silver"/>
@@ -60,9 +60,9 @@
     <origin rpy="0 0 0" xyz="-0.093 -0.0 -0.0385"/>
     <geometry>
-      <mesh filename="package://nightmare_description/meshes/leg_3_coxa_1.stl" scale="0.001 0.001 0.001"/>
-    </geometry>
-  </collision>
-</link>
-<link name="leg_4_coxa_1">
+      <mesh filename="package://nightmare_description/meshes/leg_2_coxa_1.stl" scale="0.001 0.001 0.001"/>
+    </geometry>
+  </collision>
+</link>
+<link name="leg_1_coxa_1">
   <inertial>
     <origin rpy="0 0 0" xyz="0.02405203401918829 0.02405203542330879 -0.020500001712213764"/>
@@ -73,5 +73,5 @@
     <origin rpy="0 0 0" xyz="-0.068335 -0.078335 -0.0385"/>
     <geometry>
-      <mesh filename="package://nightmare_description/meshes/leg_4_coxa_1.stl" scale="0.001 0.001 0.001"/>
+      <mesh filename="package://nightmare_description/meshes/leg_1_coxa_1.stl" scale="0.001 0.001 0.001"/>
     </geometry>
     <material name="silver"/>
@@ -80,9 +80,9 @@
     <origin rpy="0 0 0" xyz="-0.068335 -0.078335 -0.0385"/>
     <geometry>
-      <mesh filename="package://nightmare_description/meshes/leg_4_coxa_1.stl" scale="0.001 0.001 0.001"/>
-    </geometry>
-  </collision>
-</link>
-<link name="leg_5_coxa_1">
+      <mesh filename="package://nightmare_description/meshes/leg_1_coxa_1.stl" scale="0.001 0.001 0.001"/>
+    </geometry>
+  </collision>
+</link>
+<link name="leg_6_coxa_1">
   <inertial>
     <origin rpy="0 0 0" xyz="-0.02405203564458211 0.024052033797916067 -0.02050000171221522"/>
@@ -93,5 +93,5 @@
     <origin rpy="0 0 0" xyz="0.068335 -0.078335 -0.0385"/>
     <geometry>
-      <mesh filename="package://nightmare_description/meshes/leg_5_coxa_1.stl" scale="0.001 0.001 0.001"/>
+      <mesh filename="package://nightmare_description/meshes/leg_6_coxa_1.stl" scale="0.001 0.001 0.001"/>
     </geometry>
     <material name="silver"/>
@@ -100,9 +100,9 @@
     <origin rpy="0 0 0" xyz="0.068335 -0.078335 -0.0385"/>
     <geometry>
-      <mesh filename="package://nightmare_description/meshes/leg_5_coxa_1.stl" scale="0.001 0.001 0.001"/>
-    </geometry>
-  </collision>
-</link>
-<link name="leg_6_coxa_1">
+      <mesh filename="package://nightmare_description/meshes/leg_6_coxa_1.stl" scale="0.001 0.001 0.001"/>
+    </geometry>
+  </collision>
+</link>
+<link name="leg_5_coxa_1">
   <inertial>
     <origin rpy="0 0 0" xyz="-0.03401538721464084 -1.3253429337074102e-09 -0.0205000017130063"/>
@@ -113,5 +113,5 @@
     <origin rpy="0 0 0" xyz="0.093 0.0005 -0.0385"/>
     <geometry>
-      <mesh filename="package://nightmare_description/meshes/leg_6_coxa_1.stl" scale="0.001 0.001 0.001"/>
+      <mesh filename="package://nightmare_description/meshes/leg_5_coxa_1.stl" scale="0.001 0.001 0.001"/>
     </geometry>
     <material name="silver"/>
@@ -120,9 +120,9 @@
     <origin rpy="0 0 0" xyz="0.093 0.0005 -0.0385"/>
     <geometry>
-      <mesh filename="package://nightmare_description/meshes/leg_6_coxa_1.stl" scale="0.001 0.001 0.001"/>
-    </geometry>
-  </collision>
-</link>
-<link name="leg_7_coxa_1">
+      <mesh filename="package://nightmare_description/meshes/leg_5_coxa_1.stl" scale="0.001 0.001 0.001"/>
+    </geometry>
+  </collision>
+</link>
+<link name="leg_4_coxa_1">
   <inertial>
     <origin rpy="0 0 0" xyz="-0.024052033984224647 -0.024052036049472092 -0.020500001713658775"/>
@@ -133,5 +133,5 @@
     <origin rpy="0 0 0" xyz="0.068335 0.078335 -0.0385"/>
     <geometry>
-      <mesh filename="package://nightmare_description/meshes/leg_7_coxa_1.stl" scale="0.001 0.001 0.001"/>
+      <mesh filename="package://nightmare_description/meshes/leg_4_coxa_1.stl" scale="0.001 0.001 0.001"/>
     </geometry>
     <material name="silver"/>
@@ -140,9 +140,9 @@
     <origin rpy="0 0 0" xyz="0.068335 0.078335 -0.0385"/>
     <geometry>
-      <mesh filename="package://nightmare_description/meshes/leg_7_coxa_1.stl" scale="0.001 0.001 0.001"/>
-    </geometry>
-  </collision>
-</link>
-<link name="leg_2_femur_1">
+      <mesh filename="package://nightmare_description/meshes/leg_4_coxa_1.stl" scale="0.001 0.001 0.001"/>
+    </geometry>
+  </collision>
+</link>
+<link name="leg_3_femur_1">
   <inertial>
     <origin rpy="0 0 0" xyz="0.002811166294498485 -0.03199817277076898 -2.644789265403985e-05"/>
@@ -153,5 +153,5 @@
     <origin rpy="0 0 0" xyz="-0.130935 0.111944 -0.018"/>
     <geometry>
-      <mesh filename="package://nightmare_description/meshes/leg_2_femur_1.stl" scale="0.001 0.001 0.001"/>
+      <mesh filename="package://nightmare_description/meshes/leg_3_femur_1.stl" scale="0.001 0.001 0.001"/>
     </geometry>
     <material name="silver"/>
@@ -160,9 +160,9 @@
     <origin rpy="0 0 0" xyz="-0.130935 0.111944 -0.018"/>
     <geometry>
-      <mesh filename="package://nightmare_description/meshes/leg_2_femur_1.stl" scale="0.001 0.001 0.001"/>
-    </geometry>
-  </collision>
-</link>
-<link name="leg_3_femur_1">
+      <mesh filename="package://nightmare_description/meshes/leg_3_femur_1.stl" scale="0.001 0.001 0.001"/>
+    </geometry>
+  </collision>
+</link>
+<link name="leg_2_femur_1">
   <inertial>
     <origin rpy="0 0 0" xyz="0.024613629490825878 -0.02063859750853185 -2.6447892664531458e-05"/>
@@ -173,5 +173,5 @@
     <origin rpy="0 0 0" xyz="-0.161031 -0.0205 -0.018"/>
     <geometry>
-      <mesh filename="package://nightmare_description/meshes/leg_3_femur_1.stl" scale="0.001 0.001 0.001"/>
+      <mesh filename="package://nightmare_description/meshes/leg_2_femur_1.stl" scale="0.001 0.001 0.001"/>
     </geometry>
     <material name="silver"/>
@@ -180,9 +180,9 @@
     <origin rpy="0 0 0" xyz="-0.161031 -0.0205 -0.018"/>
     <geometry>
-      <mesh filename="package://nightmare_description/meshes/leg_3_femur_1.stl" scale="0.001 0.001 0.001"/>
-    </geometry>
-  </collision>
-</link>
-<link name="leg_4_femur_1">
+      <mesh filename="package://nightmare_description/meshes/leg_2_femur_1.stl" scale="0.001 0.001 0.001"/>
+    </geometry>
+  </collision>
+</link>
+<link name="leg_1_femur_1">
   <inertial>
     <origin rpy="0 0 0" xyz="0.031998172770773436 0.0028111662944979576 -2.6447892665853318e-05"/>
@@ -193,5 +193,5 @@
     <origin rpy="0 0 0" xyz="-0.101944 -0.140935 -0.018"/>
     <geometry>
-      <mesh filename="package://nightmare_description/meshes/leg_4_femur_1.stl" scale="0.001 0.001 0.001"/>
+      <mesh filename="package://nightmare_description/meshes/leg_1_femur_1.stl" scale="0.001 0.001 0.001"/>
     </geometry>
     <material name="silver"/>
@@ -200,9 +200,9 @@
     <origin rpy="0 0 0" xyz="-0.101944 -0.140935 -0.018"/>
     <geometry>
-      <mesh filename="package://nightmare_description/meshes/leg_4_femur_1.stl" scale="0.001 0.001 0.001"/>
-    </geometry>
-  </collision>
-</link>
-<link name="leg_5_femur_1">
+      <mesh filename="package://nightmare_description/meshes/leg_1_femur_1.stl" scale="0.001 0.001 0.001"/>
+    </geometry>
+  </collision>
+</link>
+<link name="leg_6_femur_1">
   <inertial>
     <origin rpy="0 0 0" xyz="-0.0318021665157692 0.0030071725494985047 -2.6447892670266454e-05"/>
@@ -213,5 +213,5 @@
     <origin rpy="0 0 0" xyz="0.101944 -0.140935 -0.018"/>
     <geometry>
-      <mesh filename="package://nightmare_description/meshes/leg_5_femur_1.stl" scale="0.001 0.001 0.001"/>
+      <mesh filename="package://nightmare_description/meshes/leg_6_femur_1.stl" scale="0.001 0.001 0.001"/>
     </geometry>
     <material name="silver"/>
@@ -220,9 +220,9 @@
     <origin rpy="0 0 0" xyz="0.101944 -0.140935 -0.018"/>
     <geometry>
-      <mesh filename="package://nightmare_description/meshes/leg_5_femur_1.stl" scale="0.001 0.001 0.001"/>
-    </geometry>
-  </collision>
-</link>
-<link name="leg_6_femur_2">
+      <mesh filename="package://nightmare_description/meshes/leg_6_femur_1.stl" scale="0.001 0.001 0.001"/>
+    </geometry>
+  </collision>
+</link>
+<link name="leg_5_femur_2">
   <inertial>
     <origin rpy="0 0 0" xyz="-0.02461362953833532 -0.020361402859740193 -2.6447930872065817e-05"/>
@@ -233,5 +233,5 @@
     <origin rpy="0 0 0" xyz="0.161031 -0.02 -0.018"/>
     <geometry>
-      <mesh filename="package://nightmare_description/meshes/leg_6_femur_2.stl" scale="0.001 0.001 0.001"/>
+      <mesh filename="package://nightmare_description/meshes/leg_5_femur_2.stl" scale="0.001 0.001 0.001"/>
     </geometry>
     <material name="silver"/>
@@ -240,9 +240,9 @@
     <origin rpy="0 0 0" xyz="0.161031 -0.02 -0.018"/>
     <geometry>
-      <mesh filename="package://nightmare_description/meshes/leg_6_femur_2.stl" scale="0.001 0.001 0.001"/>
-    </geometry>
-  </collision>
-</link>
-<link name="leg_7_femur_2">
+      <mesh filename="package://nightmare_description/meshes/leg_5_femur_2.stl" scale="0.001 0.001 0.001"/>
+    </geometry>
+  </collision>
+</link>
+<link name="leg_4_femur_2">
   <inertial>
     <origin rpy="0 0 0" xyz="-0.0030071725439563823 -0.03180216658850006 -2.64479308710458e-05"/>
@@ -253,5 +253,5 @@
     <origin rpy="0 0 0" xyz="0.130935 0.111944 -0.018"/>
     <geometry>
-      <mesh filename="package://nightmare_description/meshes/leg_7_femur_2.stl" scale="0.001 0.001 0.001"/>
+      <mesh filename="package://nightmare_description/meshes/leg_4_femur_2.stl" scale="0.001 0.001 0.001"/>
     </geometry>
     <material name="silver"/>
@@ -260,9 +260,9 @@
     <origin rpy="0 0 0" xyz="0.130935 0.111944 -0.018"/>
     <geometry>
-      <mesh filename="package://nightmare_description/meshes/leg_7_femur_2.stl" scale="0.001 0.001 0.001"/>
-    </geometry>
-  </collision>
-</link>
-<link name="leg_2_tibia_1">
+      <mesh filename="package://nightmare_description/meshes/leg_4_femur_2.stl" scale="0.001 0.001 0.001"/>
+    </geometry>
+  </collision>
+</link>
+<link name="leg_3_tibia_1">
   <inertial>
     <origin rpy="0 0 0" xyz="0.010583537273404414 -0.039709336075938184 -9.216278552708762e-05"/>
@@ -273,5 +273,5 @@
     <origin rpy="0 0 0" xyz="-0.218903 0.199204 -0.017821"/>
     <geometry>
-      <mesh filename="package://nightmare_description/meshes/leg_2_tibia_1.stl" scale="0.001 0.001 0.001"/>
+      <mesh filename="package://nightmare_description/meshes/leg_3_tibia_1.stl" scale="0.001 0.001 0.001"/>
     </geometry>
     <material name="silver"/>
@@ -280,9 +280,9 @@
     <origin rpy="0 0 0" xyz="-0.218903 0.199204 -0.017821"/>
     <geometry>
-      <mesh filename="package://nightmare_description/meshes/leg_2_tibia_1.stl" scale="0.001 0.001 0.001"/>
-    </geometry>
-  </collision>
-</link>
-<link name="leg_3_tibia_1">
+      <mesh filename="package://nightmare_description/meshes/leg_3_tibia_1.stl" scale="0.001 0.001 0.001"/>
+    </geometry>
+  </collision>
+</link>
+<link name="leg_2_tibia_1">
   <inertial>
     <origin rpy="0 0 0" xyz="0.035562049250447536 -0.02059468417445095 -9.216278925665636e-05"/>
@@ -293,5 +293,5 @@
     <origin rpy="0 0 0" xyz="-0.284936 -0.021 -0.017821"/>
     <geometry>
-      <mesh filename="package://nightmare_description/meshes/leg_3_tibia_1.stl" scale="0.001 0.001 0.001"/>
+      <mesh filename="package://nightmare_description/meshes/leg_2_tibia_1.stl" scale="0.001 0.001 0.001"/>
     </geometry>
     <material name="silver"/>
@@ -300,9 +300,9 @@
     <origin rpy="0 0 0" xyz="-0.284936 -0.021 -0.017821"/>
     <geometry>
-      <mesh filename="package://nightmare_description/meshes/leg_3_tibia_1.stl" scale="0.001 0.001 0.001"/>
-    </geometry>
-  </collision>
-</link>
-<link name="leg_4_tibia_1">
+      <mesh filename="package://nightmare_description/meshes/leg_2_tibia_1.stl" scale="0.001 0.001 0.001"/>
+    </geometry>
+  </collision>
+</link>
+<link name="leg_1_tibia_1">
   <inertial>
     <origin rpy="0 0 0" xyz="0.03970933607594407 0.0105835372734088 -9.216278554962862e-05"/>
@@ -313,5 +313,5 @@
     <origin rpy="0 0 0" xyz="-0.189204 -0.228903 -0.017821"/>
     <geometry>
-      <mesh filename="package://nightmare_description/meshes/leg_4_tibia_1.stl" scale="0.001 0.001 0.001"/>
+      <mesh filename="package://nightmare_description/meshes/leg_1_tibia_1.stl" scale="0.001 0.001 0.001"/>
     </geometry>
     <material name="silver"/>
@@ -320,9 +320,9 @@
     <origin rpy="0 0 0" xyz="-0.189204 -0.228903 -0.017821"/>
     <geometry>
-      <mesh filename="package://nightmare_description/meshes/leg_4_tibia_1.stl" scale="0.001 0.001 0.001"/>
-    </geometry>
-  </collision>
-</link>
-<link name="leg_5_tibia_1">
+      <mesh filename="package://nightmare_description/meshes/leg_1_tibia_1.stl" scale="0.001 0.001 0.001"/>
+    </geometry>
+  </collision>
+</link>
+<link name="leg_6_tibia_1">
   <inertial>
     <origin rpy="0 0 0" xyz="-0.0395755379477529 0.010717335401596334 -9.216278555388216e-05"/>
@@ -333,5 +333,5 @@
     <origin rpy="0 0 0" xyz="0.189911 -0.228196 -0.017821"/>
     <geometry>
-      <mesh filename="package://nightmare_description/meshes/leg_5_tibia_1.stl" scale="0.001 0.001 0.001"/>
+      <mesh filename="package://nightmare_description/meshes/leg_6_tibia_1.stl" scale="0.001 0.001 0.001"/>
     </geometry>
     <material name="silver"/>
@@ -340,9 +340,9 @@
     <origin rpy="0 0 0" xyz="0.189911 -0.228196 -0.017821"/>
     <geometry>
-      <mesh filename="package://nightmare_description/meshes/leg_5_tibia_1.stl" scale="0.001 0.001 0.001"/>
-    </geometry>
-  </collision>
-</link>
-<link name="leg_6_tibia_1">
+      <mesh filename="package://nightmare_description/meshes/leg_6_tibia_1.stl" scale="0.001 0.001 0.001"/>
+    </geometry>
+  </collision>
+</link>
+<link name="leg_5_tibia_1">
   <inertial>
     <origin rpy="0 0 0" xyz="-0.03556204863358775 -0.020405315407375387 -9.21627855343804e-05"/>
@@ -353,5 +353,5 @@
     <origin rpy="0 0 0" xyz="0.284936 -0.0195 -0.017821"/>
     <geometry>
-      <mesh filename="package://nightmare_description/meshes/leg_6_tibia_1.stl" scale="0.001 0.001 0.001"/>
+      <mesh filename="package://nightmare_description/meshes/leg_5_tibia_1.stl" scale="0.001 0.001 0.001"/>
     </geometry>
     <material name="silver"/>
@@ -360,9 +360,9 @@
     <origin rpy="0 0 0" xyz="0.284936 -0.0195 -0.017821"/>
     <geometry>
-      <mesh filename="package://nightmare_description/meshes/leg_6_tibia_1.stl" scale="0.001 0.001 0.001"/>
-    </geometry>
-  </collision>
-</link>
-<link name="leg_7_tibia_2">
+      <mesh filename="package://nightmare_description/meshes/leg_5_tibia_1.stl" scale="0.001 0.001 0.001"/>
+    </geometry>
+  </collision>
+</link>
+<link name="leg_4_tibia_2">
   <inertial>
     <origin rpy="0 0 0" xyz="-0.010717335112231413 -0.03957553850675136 -9.216282043532364e-05"/>
@@ -373,5 +373,5 @@
     <origin rpy="0 0 0" xyz="0.218196 0.199911 -0.017821"/>
     <geometry>
-      <mesh filename="package://nightmare_description/meshes/leg_7_tibia_2.stl" scale="0.001 0.001 0.001"/>
+      <mesh filename="package://nightmare_description/meshes/leg_4_tibia_2.stl" scale="0.001 0.001 0.001"/>
     </geometry>
     <material name="silver"/>
@@ -380,5 +380,25 @@
     <origin rpy="0 0 0" xyz="0.218196 0.199911 -0.017821"/>
     <geometry>
-      <mesh filename="package://nightmare_description/meshes/leg_7_tibia_2.stl" scale="0.001 0.001 0.001"/>
+      <mesh filename="package://nightmare_description/meshes/leg_4_tibia_2.stl" scale="0.001 0.001 0.001"/>
+    </geometry>
+  </collision>
+</link>
+<link name="tail_link_1">
+  <inertial>
+    <origin rpy="0 0 0" xyz="5.8648452051355135e-05 -0.08077626610844917 -0.02049313021079149"/>
+    <mass value="0.34035116757413375"/>
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