Commit message: updated urdf model with new legs

File: hardware-handler/nightmare_description/urdf/nightmare.xacro (robot description, xacro)
@@ -264,124 +264,4 @@
   </collision>
 </link>
-<link name="leg_3_tibia_1">
-  <inertial>
-    <origin rpy="0 0 0" xyz="0.010583537273404414 -0.039709336075938184 -9.216278552708762e-05"/>
-    <mass value="0.42195931423012945"/>
-    <inertia ixx="0.000519" ixy="0.000464" ixz="2e-06" iyy="0.000529" iyz="-2e-06" izz="0.00101"/>
-  </inertial>
-  <visual>
-    <origin rpy="0 0 0" xyz="-0.218903 0.199204 -0.017821"/>
-    <geometry>
-      <mesh filename="package://nightmare_description/meshes/leg_3_tibia_1.stl" scale="0.001 0.001 0.001"/>
-    </geometry>
-    <material name="silver"/>
-  </visual>
-  <collision>
-    <origin rpy="0 0 0" xyz="-0.218903 0.199204 -0.017821"/>
-    <geometry>
-      <mesh filename="package://nightmare_description/meshes/leg_3_tibia_1.stl" scale="0.001 0.001 0.001"/>
-    </geometry>
-  </collision>
-</link>
-<link name="leg_2_tibia_1">
-  <inertial>
-    <origin rpy="0 0 0" xyz="0.035562049250447536 -0.02059468417445095 -9.216278925665636e-05"/>
-    <mass value="0.4219593113324877"/>
-    <inertia ixx="5.9e-05" ixy="-5e-06" ixz="3e-06" iyy="0.000988" iyz="0.0" izz="0.00101"/>
-  </inertial>
-  <visual>
-    <origin rpy="0 0 0" xyz="-0.284936 -0.021 -0.017821"/>
-    <geometry>
-      <mesh filename="package://nightmare_description/meshes/leg_2_tibia_1.stl" scale="0.001 0.001 0.001"/>
-    </geometry>
-    <material name="silver"/>
-  </visual>
-  <collision>
-    <origin rpy="0 0 0" xyz="-0.284936 -0.021 -0.017821"/>
-    <geometry>
-      <mesh filename="package://nightmare_description/meshes/leg_2_tibia_1.stl" scale="0.001 0.001 0.001"/>
-    </geometry>
-  </collision>
-</link>
-<link name="leg_1_tibia_1">
-  <inertial>
-    <origin rpy="0 0 0" xyz="0.03970933607594407 0.0105835372734088 -9.216278554962862e-05"/>
-    <mass value="0.4219593142300533"/>
-    <inertia ixx="0.000529" ixy="-0.000464" ixz="2e-06" iyy="0.000519" iyz="2e-06" izz="0.00101"/>
-  </inertial>
-  <visual>
-    <origin rpy="0 0 0" xyz="-0.189204 -0.228903 -0.017821"/>
-    <geometry>
-      <mesh filename="package://nightmare_description/meshes/leg_1_tibia_1.stl" scale="0.001 0.001 0.001"/>
-    </geometry>
-    <material name="silver"/>
-  </visual>
-  <collision>
-    <origin rpy="0 0 0" xyz="-0.189204 -0.228903 -0.017821"/>
-    <geometry>
-      <mesh filename="package://nightmare_description/meshes/leg_1_tibia_1.stl" scale="0.001 0.001 0.001"/>
-    </geometry>
-  </collision>
-</link>
-<link name="leg_6_tibia_1">
-  <inertial>
-    <origin rpy="0 0 0" xyz="-0.0395755379477529 0.010717335401596334 -9.216278555388216e-05"/>
-    <mass value="0.4219593142301195"/>
-    <inertia ixx="0.000519" ixy="0.000464" ixz="-2e-06" iyy="0.000529" iyz="2e-06" izz="0.00101"/>
-  </inertial>
-  <visual>
-    <origin rpy="0 0 0" xyz="0.189911 -0.228196 -0.017821"/>
-    <geometry>
-      <mesh filename="package://nightmare_description/meshes/leg_6_tibia_1.stl" scale="0.001 0.001 0.001"/>
-    </geometry>
-    <material name="silver"/>
-  </visual>
-  <collision>
-    <origin rpy="0 0 0" xyz="0.189911 -0.228196 -0.017821"/>
-    <geometry>
-      <mesh filename="package://nightmare_description/meshes/leg_6_tibia_1.stl" scale="0.001 0.001 0.001"/>
-    </geometry>
-  </collision>
-</link>
-<link name="leg_5_tibia_1">
-  <inertial>
-    <origin rpy="0 0 0" xyz="-0.03556204863358775 -0.020405315407375387 -9.21627855343804e-05"/>
-    <mass value="0.4219593142301098"/>
-    <inertia ixx="5.9e-05" ixy="-5e-06" ixz="-3e-06" iyy="0.000988" iyz="-0.0" izz="0.00101"/>
-  </inertial>
-  <visual>
-    <origin rpy="0 0 0" xyz="0.284936 -0.0195 -0.017821"/>
-    <geometry>
-      <mesh filename="package://nightmare_description/meshes/leg_5_tibia_1.stl" scale="0.001 0.001 0.001"/>
-    </geometry>
-    <material name="silver"/>
-  </visual>
-  <collision>
-    <origin rpy="0 0 0" xyz="0.284936 -0.0195 -0.017821"/>
-    <geometry>
-      <mesh filename="package://nightmare_description/meshes/leg_5_tibia_1.stl" scale="0.001 0.001 0.001"/>
-    </geometry>
-  </collision>
-</link>
-<link name="leg_4_tibia_2">
-  <inertial>
-    <origin rpy="0 0 0" xyz="-0.010717335112231413 -0.03957553850675136 -9.216282043532364e-05"/>
-    <mass value="0.42195931775079665"/>
-    <inertia ixx="0.000529" ixy="-0.000464" ixz="-2e-06" iyy="0.000519" iyz="-2e-06" izz="0.00101"/>
-  </inertial>
-  <visual>
-    <origin rpy="0 0 0" xyz="0.218196 0.199911 -0.017821"/>
-    <geometry>
-      <mesh filename="package://nightmare_description/meshes/leg_4_tibia_2.stl" scale="0.001 0.001 0.001"/>
-    </geometry>
-    <material name="silver"/>
-  </visual>
-  <collision>
-    <origin rpy="0 0 0" xyz="0.218196 0.199911 -0.017821"/>
-    <geometry>
-      <mesh filename="package://nightmare_description/meshes/leg_4_tibia_2.stl" scale="0.001 0.001 0.001"/>
-    </geometry>
-  </collision>
-</link>
 <link name="tail_link_1">
   <inertial>
@@ -401,4 +281,124 @@
     <geometry>
       <mesh filename="package://nightmare_description/meshes/tail_link_1.stl" scale="0.001 0.001 0.001"/>
+    </geometry>
+  </collision>
+</link>
+<link name="leg_1_tibia_2">
+  <inertial>
+    <origin rpy="0 0 0" xyz="0.04597168022169831 0.016860788290768453 0.015065036661186085"/>
+    <mass value="0.9516929282440427"/>
+    <inertia ixx="0.001279" ixy="-0.001095" ixz="-1.5e-05" iyy="0.001324" iyz="-1.8e-05" izz="0.002344"/>
+  </inertial>
+  <visual>
+    <origin rpy="0 0 0" xyz="-0.189204 -0.228903 -0.017821"/>
+    <geometry>
+      <mesh filename="package://nightmare_description/meshes/leg_1_tibia_2.stl" scale="0.001 0.001 0.001"/>
+    </geometry>
+    <material name="silver"/>
+  </visual>
+  <collision>
+    <origin rpy="0 0 0" xyz="-0.189204 -0.228903 -0.017821"/>
+    <geometry>
+      <mesh filename="package://nightmare_description/meshes/leg_1_tibia_2.stl" scale="0.001 0.001 0.001"/>
+    </geometry>
+  </collision>
+</link>
+<link name="leg_2_tibia_1">
+  <inertial>
+    <origin rpy="0 0 0" xyz="0.04442888153142993 -0.020584144796290275 0.0150650361958693"/>
+    <mass value="0.9516929282440427"/>
+    <inertia ixx="0.000206" ixy="2.2e-05" ixz="-2.3e-05" iyy="0.002396" iyz="-2e-06" izz="0.002344"/>
+  </inertial>
+  <visual>
+    <origin rpy="0 0 0" xyz="-0.284936 -0.021 -0.017821"/>
+    <geometry>
+      <mesh filename="package://nightmare_description/meshes/leg_2_tibia_1.stl" scale="0.001 0.001 0.001"/>
+    </geometry>
+    <material name="silver"/>
+  </visual>
+  <collision>
+    <origin rpy="0 0 0" xyz="-0.284936 -0.021 -0.017821"/>
+    <geometry>
+      <mesh filename="package://nightmare_description/meshes/leg_2_tibia_1.stl" scale="0.001 0.001 0.001"/>
+    </geometry>
+  </collision>
+</link>
+<link name="leg_3_tibia_1">
+  <inertial>
+    <origin rpy="0 0 0" xyz="0.016860788832001927 -0.045971679856765535 0.015065036195894974"/>
+    <mass value="0.9516929282440427"/>
+    <inertia ixx="0.001324" ixy="0.001095" ixz="-1.8e-05" iyy="0.001279" iyz="1.5e-05" izz="0.002344"/>
+  </inertial>
+  <visual>
+    <origin rpy="0 0 0" xyz="-0.218903 0.199204 -0.017821"/>
+    <geometry>
+      <mesh filename="package://nightmare_description/meshes/leg_3_tibia_1.stl" scale="0.001 0.001 0.001"/>
+    </geometry>
+    <material name="silver"/>
+  </visual>
+  <collision>
+    <origin rpy="0 0 0" xyz="-0.218903 0.199204 -0.017821"/>
+    <geometry>
+      <mesh filename="package://nightmare_description/meshes/leg_3_tibia_1.stl" scale="0.001 0.001 0.001"/>
+    </geometry>
+  </collision>
+</link>
+<link name="leg_4_tibia_1">
+  <inertial>
+    <origin rpy="0 0 0" xyz="-0.016979679635497652 -0.04585278905326559 0.015065036195897347"/>
+    <mass value="0.9516929282440427"/>
+    <inertia ixx="0.001279" ixy="-0.001095" ixz="1.5e-05" iyy="0.001324" iyz="1.8e-05" izz="0.002344"/>
+  </inertial>
+  <visual>
+    <origin rpy="0 0 0" xyz="0.218196 0.199911 -0.017821"/>
+    <geometry>
+      <mesh filename="package://nightmare_description/meshes/leg_4_tibia_1.stl" scale="0.001 0.001 0.001"/>
+    </geometry>
+    <material name="silver"/>
+  </visual>
+  <collision>
+    <origin rpy="0 0 0" xyz="0.218196 0.199911 -0.017821"/>
+    <geometry>
+      <mesh filename="package://nightmare_description/meshes/leg_4_tibia_1.stl" scale="0.001 0.001 0.001"/>
+    </geometry>
+  </collision>
+</link>
+<link name="leg_5_tibia_1">
+  <inertial>
+    <origin rpy="0 0 0" xyz="-0.04442888153142355 -0.02041585551662712 0.015065036195890901"/>
+    <mass value="0.9516929282440427"/>
+    <inertia ixx="0.000206" ixy="2.2e-05" ixz="2.3e-05" iyy="0.002396" iyz="2e-06" izz="0.002344"/>
+  </inertial>
+  <visual>
+    <origin rpy="0 0 0" xyz="0.284936 -0.0195 -0.017821"/>
+    <geometry>
+      <mesh filename="package://nightmare_description/meshes/leg_5_tibia_1.stl" scale="0.001 0.001 0.001"/>
+    </geometry>
+    <material name="silver"/>
+  </visual>
+  <collision>
+    <origin rpy="0 0 0" xyz="0.284936 -0.0195 -0.017821"/>
+    <geometry>
+      <mesh filename="package://nightmare_description/meshes/leg_5_tibia_1.stl" scale="0.001 0.001 0.001"/>
+    </geometry>
+  </collision>
+</link>
+<link name="leg_6_tibia_1">
+  <inertial>
+    <origin rpy="0 0 0" xyz="-0.0458527886001843 0.01697968008857778 0.015065036195873956"/>
+    <mass value="0.9516929282440427"/>
+    <inertia ixx="0.001324" ixy="0.001095" ixz="1.8e-05" iyy="0.001279" iyz="-1.5e-05" izz="0.002344"/>
+  </inertial>
+  <visual>
+    <origin rpy="0 0 0" xyz="0.189911 -0.228196 -0.017821"/>
+    <geometry>
+      <mesh filename="package://nightmare_description/meshes/leg_6_tibia_1.stl" scale="0.001 0.001 0.001"/>
+    </geometry>
+    <material name="silver"/>
+  </visual>
+  <collision>
+    <origin rpy="0 0 0" xyz="0.189911 -0.228196 -0.017821"/>
+    <geometry>
+      <mesh filename="package://nightmare_description/meshes/leg_6_tibia_1.stl" scale="0.001 0.001 0.001"/>
     </geometry>
   </collision>
@@ -476,4 +476,22 @@
   <axis xyz="-0.707107 0.707107 0.0"/>
 </joint>
+<joint name="Rev121" type="continuous">
+  <origin rpy="0 0 0" xyz="0.0 -0.113 0.0385"/>
+  <parent link="base_link"/>
+  <child link="tail_link_1"/>
+  <axis xyz="-0.0 0.0 -1.0"/>
+</joint>
+<joint name="Rev117" type="continuous">
+  <origin rpy="0 0 0" xyz="0.08726 0.087968 -0.000179"/>
+  <parent link="leg_1_femur_1"/>
+  <child link="leg_1_tibia_2"/>
+  <axis xyz="0.707107 -0.707107 -0.0"/>
+</joint>
+<joint name="Rev116" type="continuous">
+  <origin rpy="0 0 0" xyz="0.123905 0.0005 -0.000179"/>
+  <parent link="leg_2_femur_1"/>
+  <child link="leg_2_tibia_1"/>
+  <axis xyz="0.0 -1.0 -0.0"/>
+</joint>
 <joint name="Rev115" type="continuous">
   <origin rpy="0 0 0" xyz="0.087968 -0.08726 -0.000179"/>
@@ -482,15 +500,15 @@
   <axis xyz="-0.707107 -0.707107 -0.0"/>
 </joint>
-<joint name="Rev116" type="continuous">
-  <origin rpy="0 0 0" xyz="0.123905 0.0005 -0.000179"/>
-  <parent link="leg_2_femur_1"/>
-  <child link="leg_2_tibia_1"/>
-  <axis xyz="0.0 -1.0 -0.0"/>
-</joint>
-<joint name="Rev117" type="continuous">
-  <origin rpy="0 0 0" xyz="0.08726 0.087968 -0.000179"/>
-  <parent link="leg_1_femur_1"/>
-  <child link="leg_1_tibia_1"/>
-  <axis xyz="0.707107 -0.707107 -0.0"/>
+<joint name="Rev120" type="continuous">
+  <origin rpy="0 0 0" xyz="-0.087261 -0.087967 -0.000179"/>
+  <parent link="leg_4_femur_2"/>
+  <child link="leg_4_tibia_1"/>
+  <axis xyz="-0.707107 0.707107 -0.0"/>
+</joint>
+<joint name="Rev119" type="continuous">
+  <origin rpy="0 0 0" xyz="-0.123905 -0.0005 -0.000179"/>
+  <parent link="leg_5_femur_2"/>
+  <child link="leg_5_tibia_1"/>
+  <axis xyz="0.0 1.0 -0.0"/>
 </joint>
 <joint name="Rev118" type="continuous">
@@ -500,21 +518,3 @@
   <axis xyz="0.707107 0.707107 -0.0"/>
 </joint>
-<joint name="Rev119" type="continuous">
-  <origin rpy="0 0 0" xyz="-0.123905 -0.0005 -0.000179"/>
-  <parent link="leg_5_femur_2"/>
-  <child link="leg_5_tibia_1"/>
-  <axis xyz="0.0 1.0 -0.0"/>
-</joint>
-<joint name="Rev120" type="continuous">
-  <origin rpy="0 0 0" xyz="-0.087261 -0.087967 -0.000179"/>
-  <parent link="leg_4_femur_2"/>
-  <child link="leg_4_tibia_2"/>
-  <axis xyz="-0.707107 0.707107 -0.0"/>
-</joint>
-<joint name="Rev121" type="continuous">
-  <origin rpy="0 0 0" xyz="0.0 -0.113 0.0385"/>
-  <parent link="base_link"/>
-  <child link="tail_link_1"/>
-  <axis xyz="-0.0 0.0 -1.0"/>
-</joint>
 </robot>

Commit message: added more human friendly names

File: hardware-handler/nightmare_description/urdf/nightmare.xacro (robot description, xacro)
@@ -404,5 +404,5 @@
   </collision>
 </link>
-<joint name="Rev103" type="continuous">
+<joint name="leg3coxa" type="continuous">
   <origin rpy="0 0 0" xyz="0.068335 -0.078335 0.0385"/>
   <parent link="base_link"/>
@@ -410,5 +410,5 @@
   <axis xyz="-0.0 -0.0 -1.0"/>
 </joint>
-<joint name="Rev104" type="continuous">
+<joint name="leg2coxa" type="continuous">
   <origin rpy="0 0 0" xyz="0.093 0.0 0.0385"/>
   <parent link="base_link"/>
@@ -416,5 +416,5 @@
   <axis xyz="-0.0 0.0 -1.0"/>
 </joint>
-<joint name="Rev105" type="continuous">
+<joint name="leg1coxa" type="continuous">
   <origin rpy="0 0 0" xyz="0.068335 0.078335 0.0385"/>
   <parent link="base_link"/>
@@ -422,5 +422,5 @@
   <axis xyz="0.0 -0.0 -1.0"/>
 </joint>
-<joint name="Rev106" type="continuous">
+<joint name="leg6coxa" type="continuous">
   <origin rpy="0 0 0" xyz="-0.068335 0.078335 0.0385"/>
   <parent link="base_link"/>
@@ -428,5 +428,5 @@
   <axis xyz="0.0 -0.0 -1.0"/>
 </joint>
-<joint name="Rev107" type="continuous">
+<joint name="leg5coxa" type="continuous">
   <origin rpy="0 0 0" xyz="-0.093 -0.0005 0.0385"/>
   <parent link="base_link"/>
@@ -434,5 +434,5 @@
   <axis xyz="-0.0 0.0 -1.0"/>
 </joint>
-<joint name="Rev108" type="continuous">
+<joint name="leg4coxa" type="continuous">
   <origin rpy="0 0 0" xyz="-0.068335 -0.078335 0.0385"/>
   <parent link="base_link"/>
@@ -440,5 +440,5 @@
   <axis xyz="-0.0 0.0 -1.0"/>
 </joint>
-<joint name="Rev109" type="continuous">
+<joint name="leg3femur" type="continuous">
   <origin rpy="0 0 0" xyz="0.0626 -0.033609 -0.0205"/>
   <parent link="leg_3_coxa_1"/>
@@ -446,5 +446,5 @@
   <axis xyz="-0.707107 -0.707107 0.0"/>
 </joint>
-<joint name="Rev110" type="continuous">
+<joint name="leg2femur" type="continuous">
   <origin rpy="0 0 0" xyz="0.068031 0.0205 -0.0205"/>
   <parent link="leg_2_coxa_1"/>
@@ -452,5 +452,5 @@
   <axis xyz="-0.0 -1.0 -0.0"/>
 </joint>
-<joint name="Rev111" type="continuous">
+<joint name="leg1femur" type="continuous">
   <origin rpy="0 0 0" xyz="0.033609 0.0626 -0.0205"/>
   <parent link="leg_1_coxa_1"/>
@@ -458,5 +458,5 @@
   <axis xyz="0.707107 -0.707107 0.0"/>
 </joint>
-<joint name="Rev112" type="continuous">
+<joint name="leg6femur" type="continuous">
   <origin rpy="0 0 0" xyz="-0.033609 0.0626 -0.0205"/>
   <parent link="leg_6_coxa_1"/>
@@ -464,5 +464,5 @@
   <axis xyz="0.707107 0.707107 -0.0"/>
 </joint>
-<joint name="Rev113" type="continuous">
+<joint name="leg5femur" type="continuous">
   <origin rpy="0 0 0" xyz="-0.068031 0.0205 -0.0205"/>
   <parent link="leg_5_coxa_1"/>
@@ -470,5 +470,5 @@
   <axis xyz="0.0 1.0 0.0"/>
 </joint>
-<joint name="Rev114" type="continuous">
+<joint name="leg4femur" type="continuous">
   <origin rpy="0 0 0" xyz="-0.0626 -0.033609 -0.0205"/>
   <parent link="leg_4_coxa_1"/>
@@ -476,5 +476,5 @@
   <axis xyz="-0.707107 0.707107 0.0"/>
 </joint>
-<joint name="Rev121" type="continuous">
+<joint name="tail_joint" type="continuous">
   <origin rpy="0 0 0" xyz="0.0 -0.113 0.0385"/>
   <parent link="base_link"/>
@@ -482,5 +482,5 @@
   <axis xyz="-0.0 0.0 -1.0"/>
 </joint>
-<joint name="Rev117" type="continuous">
+<joint name="leg1tibia" type="continuous">
   <origin rpy="0 0 0" xyz="0.08726 0.087968 -0.000179"/>
   <parent link="leg_1_femur_1"/>
@@ -488,5 +488,5 @@
   <axis xyz="0.707107 -0.707107 -0.0"/>
 </joint>
-<joint name="Rev116" type="continuous">
+<joint name="leg2tibia" type="continuous">
   <origin rpy="0 0 0" xyz="0.123905 0.0005 -0.000179"/>
   <parent link="leg_2_femur_1"/>
@@ -494,5 +494,5 @@
   <axis xyz="0.0 -1.0 -0.0"/>
 </joint>
-<joint name="Rev115" type="continuous">
+<joint name="leg3tibia" type="continuous">
   <origin rpy="0 0 0" xyz="0.087968 -0.08726 -0.000179"/>
   <parent link="leg_3_femur_1"/>
@@ -500,5 +500,5 @@
   <axis xyz="-0.707107 -0.707107 -0.0"/>
 </joint>
-<joint name="Rev120" type="continuous">
+<joint name="leg4tibia" type="continuous">
   <origin rpy="0 0 0" xyz="-0.087261 -0.087967 -0.000179"/>
   <parent link="leg_4_femur_2"/>
@@ -506,5 +506,5 @@
   <axis xyz="-0.707107 0.707107 -0.0"/>
 </joint>
-<joint name="Rev119" type="continuous">
+<joint name="leg5tibia" type="continuous">
   <origin rpy="0 0 0" xyz="-0.123905 -0.0005 -0.000179"/>
   <parent link="leg_5_femur_2"/>
@@ -512,5 +512,5 @@
   <axis xyz="0.0 1.0 -0.0"/>
 </joint>
-<joint name="Rev118" type="continuous">
+<joint name="leg6tibia" type="continuous">
   <origin rpy="0 0 0" xyz="-0.087967 0.087261 -0.000179"/>
   <parent link="leg_6_femur_1"/>

Commit message: fixed base_link has inertia: inertia is no more

File: hardware-handler/nightmare_description/urdf/nightmare.xacro (robot description, xacro)
@@ -5,4 +5,6 @@
 <xacro:include filename="$(find nightmare_description)/urdf/nightmare.gazebo" />
 <link name="base_link">
+</link>
+<link name="body_link">
   <inertial>
     <origin rpy="0 0 0" xyz="0.00027642737085348105 0.010613740030603296 0.02249920074743168"/>
@@ -404,7 +406,12 @@
   </collision>
 </link>
+<joint name="base2body" type="fixed">
+  <origin rpy="0 0 0" xyz="0 0 0"/>
+  <parent link="base_link"/>
+  <child link="body_link"/>
+</joint>
 <joint name="leg3coxa" type="continuous">
   <origin rpy="0 0 0" xyz="0.068335 -0.078335 0.0385"/>
-  <parent link="base_link"/>
+  <parent link="body_link"/>
   <child link="leg_3_coxa_1"/>
   <axis xyz="-0.0 -0.0 -1.0"/>
@@ -412,5 +419,5 @@
 <joint name="leg2coxa" type="continuous">
   <origin rpy="0 0 0" xyz="0.093 0.0 0.0385"/>
-  <parent link="base_link"/>
+  <parent link="body_link"/>
   <child link="leg_2_coxa_1"/>
   <axis xyz="-0.0 0.0 -1.0"/>
@@ -418,5 +425,5 @@
 <joint name="leg1coxa" type="continuous">
   <origin rpy="0 0 0" xyz="0.068335 0.078335 0.0385"/>
-  <parent link="base_link"/>
+  <parent link="body_link"/>
   <child link="leg_1_coxa_1"/>
   <axis xyz="0.0 -0.0 -1.0"/>
@@ -424,5 +431,5 @@
 <joint name="leg6coxa" type="continuous">
   <origin rpy="0 0 0" xyz="-0.068335 0.078335 0.0385"/>
-  <parent link="base_link"/>
+  <parent link="body_link"/>
   <child link="leg_6_coxa_1"/>
   <axis xyz="0.0 -0.0 -1.0"/>
@@ -430,5 +437,5 @@
 <joint name="leg5coxa" type="continuous">
   <origin rpy="0 0 0" xyz="-0.093 -0.0005 0.0385"/>
-  <parent link="base_link"/>
+  <parent link="body_link"/>
   <child link="leg_5_coxa_1"/>
   <axis xyz="-0.0 0.0 -1.0"/>
@@ -436,5 +443,5 @@
 <joint name="leg4coxa" type="continuous">
   <origin rpy="0 0 0" xyz="-0.068335 -0.078335 0.0385"/>
-  <parent link="base_link"/>
+  <parent link="body_link"/>
   <child link="leg_4_coxa_1"/>
   <axis xyz="-0.0 0.0 -1.0"/>
@@ -478,5 +485,5 @@
 <joint name="tail_joint" type="continuous">
   <origin rpy="0 0 0" xyz="0.0 -0.113 0.0385"/>
-  <parent link="base_link"/>
+  <parent link="body_link"/>
   <child link="tail_link_1"/>
   <axis xyz="-0.0 0.0 -1.0"/>
